File: PCB Files (WIP)/Moth.kicad_pcb (KiCad board)
At the start: 2 copper layers, 239 x 118.3 mm, 62 parts, among them J1 USB C Connector, J2 JTAG_TC2030, J3 Left Ribbon, J4 Right Ribbon, SW1 Boot, U1 XC6206, U2 USBLC6-2SC6, U3 RP2040, U4 W25Q128JVS, X1 X, Y1 12MHz, Y2 Y

Commit message: Add files via upload
Parts:
- moved J3 7.29 mm to (166.3, 79.9), turned to 90 degrees
- moved J4 6.77 mm to (130.1, 79.8), turned to -90 degrees
Connections:
- J3 pad 1: R RIBBON1 -> unconnected-(J3-Pin_1-Pad1)
- J3 pad 10: C_DN RIBBON1 -> A RIBBON1
- J3 pad 11: A RIBBON1 -> C_DN RIBBON1
- J3 pad 12: C_LT RIBBON1 -> C_DN RIBBON1
- J3 pad 13: C_UP RIBBON1 -> UP RIBBON1
- J3 pad 14: GND RIBBON1 -> MS RIBBON1
- J3 pad 15: unconnected-(J3-Pin_15-Pad15) -> Z RIBBON1
- J3 pad 16: unconnected-(J3-Pin_16-Pad16) -> LS RIBBON1
- J3 pad 17: unconnected-(J3-Pin_17-Pad17) -> X RIBBON1
- J3 pad 18: unconnected-(J3-Pin_18-Pad18) -> Y RIBBON1
- J3 pad 19: unconnected-(J3-Pin_19-Pad19) -> B RIBBON1
- J3 pad 2: B RIBBON1 -> unconnected-(J3-Pin_2-Pad2)
- J3 pad 20: unconnected-(J3-Pin_20-Pad20) -> R RIBBON1
- J3 pad 3: Y RIBBON1 -> unconnected-(J3-Pin_3-Pad3)
- J3 pad 4: X RIBBON1 -> unconnected-(J3-Pin_4-Pad4)
- J3 pad 5: LS RIBBON1 -> unconnected-(J3-Pin_5-Pad5)
- J3 pad 6: Z RIBBON1 -> unconnected-(J3-Pin_6-Pad6)
- J3 pad 7: MS RIBBON1 -> GND RIBBON1
- J3 pad 8: UP RIBBON1 -> C_UP RIBBON1
- J3 pad 9: C_RT RIBBON1 -> C_LT RIBBON1
- U3 pad 27: C_RT RIBBON1 -> C_DN RIBBON1
Routing:
- net C_RT RIBBON1: track 77.8 -> 0.00 mm
- net C_DN RIBBON1: track 93.2 -> 165.9 mm
- net MS: track 142.4 -> 102.8 mm, vias 0 -> 2
- net X: track 78.4 -> 52.8 mm
- net GND: track 88.8 -> 113.6 mm
- net L: track 121.3 -> 96.9 mm
- net LS: track 122.8 -> 99.3 mm
- net C_UP: track 49.2 -> 69.1 mm, vias 0 -> 2
- net R: track 30.7 -> 41.9 mm, vias 0 -> 2
- net START: track 77.8 -> 67.1 mm
- net Y: track 63.6 -> 74.0 mm, vias 0 -> 2
- net C_LT: track 70.7 -> 81.0 mm, vias 0 -> 2
- net B: track 44.2 -> 35.2 mm, vias 1 -> 2
- net UP: track 122.2 -> 129.1 mm
- net A: track 85.6 -> 80.8 mm, vias 0 -> 2
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
Commit message: Reconfigured PCB, closer to completion.
Parts:
- removed D2: Schottky Diode, Diode_SMD:D_SOD-123
- removed F1: 500 mA, Fuse:Fuse_1206_3216Metric
- removed R12: R, moth footprints:SW_Gateron_LowProfile_HotSwap_THT
- removed R2, R3: 5.1k, Resistor_SMD:R_0402_1005Metric
- added J5: Right Ribbon, moth footprints:FPC-05F-30PH20, F.Cu at (129.4, 79.1)
- J1: value USB C Connector -> Conn_01x02; footprint footprints:TYPE-C_24P_QCHT -> Connector_PinHeader_2.54mm:PinHeader_1x02_P2.54mm_Vertical
- J3: value Left Ribbon -> DuPont Connector; footprint moth footprints:FPC-05F-30PH20 -> Connector_PinHeader_2.54mm:PinHeader_1x06_P2.54mm_Vertical
- J4: value Right Ribbon -> Left Ribbon
- R1: value 1M -> R; footprint Resistor_SMD:R_0603_1608Metric -> moth footprints:SW_Gateron_LowProfile_HotSwap_THT; moved to B.Cu
- R4: value 10k -> 470
- U2: value USBLC6-2SC6 -> X05A26H12G; footprint Package_TO_SOT_SMD:SOT-23-6 -> footprint:FPC-SMD_X05A26H12G
- U3: footprint footprints:RP2040-QFN-56 -> qw-footprints:RP2040-QFN-56
- moved R1 148.6 mm to (111.8, 62.1), turned to 180 degrees
- moved J3 45.8 mm to (209.0, 63.2), turned to -90 degrees
- moved U2 35.4 mm to (215.0, 84.1)
- moved J4 24.3 mm to (154.4, 79.1), turned to 90 degrees
- moved D3 20.0 mm to (205.6, 131.8)
- moved R4 19.9 mm to (205.6, 129.2)
- moved MY1 16.7 mm to (158.7, 145.2)
- moved LEFT1 16.7 mm to (220.1, 70.3)
- moved L1 16.7 mm to (241.8, 74.9), turned to 180 degrees
- moved DOWN1 16.7 mm to (198.1, 73.4)
- moved MX1 16.7 mm to (176.2, 131.2)
- moved START1 16.7 mm to (189.5, 52.9)
- moved RIGHT1 16.7 mm to (178.6, 83.8)
- moved J1 14.8 mm to (238.1, 107.9), turned to 180 degrees
- moved C7 13.1 mm to (200.1, 112.5)
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Connections:
- C1 pad 2: +3V3 -> 3vDiode
- C10 pad 1: +3V3 -> 3vDiode
- C11 pad 1: +3V3 -> 3vDiode
- C12 pad 1: +3V3 -> 3vDiode
- C13 pad 1: +3V3 -> 3vDiode
- C14 pad 1: +3V3 -> 3vDiode
- C15 pad 1: +3V3 -> 3vDiode
- C16 pad 1: +3V3 -> 3vDiode
- C17 pad 1: +3V3 -> 3vDiode
- C3 pad 1: +3V3 -> 3vDiode
- C9 pad 1: +3V3 -> 3vDiode
- D1 pad 1: +3V3 -> 3vDiode
- J2 pad 1: +3V3 -> 3vDiode
- J3 pad 1: unconnected-(J3-Pin_1-Pad1) -> GND
- J3 pad 2: unconnected-(J3-Pin_2-Pad2) -> +5V
- J3 pad 3: unconnected-(J3-Pin_3-Pad3) -> D+
- J3 pad 4: unconnected-(J3-Pin_4-Pad4) -> D-
- J3 pad 5: unconnected-(J3-Pin_5-Pad5) -> DATA
- J3 pad 6: unconnected-(J3-Pin_6-Pad6) -> 3vDiode
- J4 pad 1: R -> unconnected-(J4-Pin_1-Pad1)
- J4 pad 10: C_DN -> A RIBBON
- J4 pad 11: A -> C_DN RIBBON
- J4 pad 12: C_LT -> C_RT RIBBON
- J4 pad 13: C_UP -> UP RIBBON
- J4 pad 14: GND -> MS RIBBON
- J4 pad 15: unconnected-(J4-Pin_15-Pad15) -> Z RIBBON
- J4 pad 16: unconnected-(J4-Pin_16-Pad16) -> LS RIBBON
- J4 pad 17: unconnected-(J4-Pin_17-Pad17) -> X RIBBON
- J4 pad 18: unconnected-(J4-Pin_18-Pad18) -> Y RIBBON
- J4 pad 19: unconnected-(J4-Pin_19-Pad19) -> B RIBBON
- J4 pad 2: B -> unconnected-(J4-Pin_2-Pad2)
- J4 pad 20: unconnected-(J4-Pin_20-Pad20) -> R RIBBON
- J4 pad 3: Y -> unconnected-(J4-Pin_3-Pad3)
- J4 pad 4: X -> unconnected-(J4-Pin_4-Pad4)
- J4 pad 5: LS -> unconnected-(J4-Pin_5-Pad5)
- J4 pad 6: Z -> unconnected-(J4-Pin_6-Pad6)
- J4 pad 7: MS -> GND
- J4 pad 8: UP -> C_UP RIBBON
- J4 pad 9: C_RT -> C_LT RIBBON
- R1 pad 1: GND -> R
- R1 pad 2: Net-(J1-SHIELD) -> GND
- R7 pad 1: +3V3 -> 3vDiode
- U2 pad 1: DBUS+ -> 3vDiode
- U2 pad 2: GND -> 3vDiode
- U2 pad 3: DBUS- -> DATA
- U2 pad 4: D- -> DATA
- U2 pad 5: +5V -> D-
- U2 pad 6: D+ -> D-
- U3 pad 1: +3V3 -> 3vDiode
- U3 pad 10: +3V3 -> 3vDiode
- U3 pad 15: C_UP RIBBON1 -> C_UP RIBBON
- U3 pad 16: C_LT RIBBON1 -> C_LT RIBBON
- U3 pad 17: A RIBBON1 -> A RIBBON
- U3 pad 18: C_DN RIBBON1 -> C_DN RIBBON
- U3 pad 22: +3V3 -> 3vDiode
- U3 pad 27: C_DN RIBBON1 -> C_RT RIBBON
- U3 pad 28: UP RIBBON1 -> UP RIBBON
- U3 pad 29: MS RIBBON1 -> MS RIBBON
- U3 pad 30: Z RIBBON1 -> Z RIBBON
- U3 pad 31: LS RIBBON1 -> LS RIBBON
- U3 pad 32: X RIBBON1 -> X RIBBON
- U3 pad 33: +3V3 -> 3vDiode
- U3 pad 34: Y RIBBON1 -> Y RIBBON
- U3 pad 38: B RIBBON1 -> B RIBBON
- U3 pad 39: R RIBBON1 -> R RIBBON
- U3 pad 42: +3V3 -> 3vDiode
- U3 pad 43: +3V3 -> 3vDiode
- U3 pad 44: +3V3 -> 3vDiode
- U3 pad 48: +3V3 -> 3vDiode
- U3 pad 49: +3V3 -> 3vDiode
- U4 pad 8: +3V3 -> 3vDiode
Routing:
- net C_DN RIBBON1: track 165.9 -> 0.00 mm
- net 3vDiode: track 0.00 -> 142.2 mm, vias 0 -> 7
- net R RIBBON: track 0.00 -> 114.1 mm
- net B RIBBON: track 0.00 -> 113.5 mm
- net X RIBBON: track 0.00 -> 112.4 mm
- net Y RIBBON: track 0.00 -> 112.4 mm
- net LS RIBBON: track 0.00 -> 111.7 mm
- net C_RT RIBBON: track 0.00 -> 111.3 mm
- net Z RIBBON: track 0.00 -> 111.0 mm
- net UP RIBBON: track 0.00 -> 110.8 mm
- net MS RIBBON: track 0.00 -> 110.2 mm
- net C_LT RIBBON: track 0.00 -> 91.6 mm
- net C_UP RIBBON: track 0.00 -> 91.5 mm
- net A RIBBON: track 0.00 -> 91.5 mm
- net C_DN RIBBON: track 0.00 -> 91.3 mm
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- added copper zone on F.Cu, net 3vDiode
- removed copper zone on F.Cu, net +3V3
Other:
- board size 239 x 118.3 mm -> 220.6 x 118.4 mm
- board text added: "3v3 DATA D- D+ 5+ GND"
- board text added: "A"
- board text added: "B"
- board text added: "Boot"
- board text added: "C-DOWN"
- board text added: "C-LEFT"
- board text added: "C-RIGHT"
- board text added: "C-UP"
- board text added: "DOWN"
- board text added: "L"
- board text added: "LEFT"
- board text added: "LS"
- board text added: "MS"
- board text added: "MX"
- board text added: "MY"
- board text added: "R"
- board text added: "RANA MOTH BY RANA LABS"
- board text added: "RIGHT"
- board text added: "START"
- board text added: "UP"
- board text added: "X"
- board text added: "Y"
- board text added: "Z"

Commit message: Completed PCB pending review
Parts:
- A1, B1, C_DOWN1, C_LEFT1, C_RIGHT1, C_UP1, L1, LEFT1, LS1, MS1, MX1, MY1, R1, RIGHT1, START1, UP1, X1, Y2, Z1: footprint moth footprints:SW_Gateron_LowProfile_HotSwap_THT -> Box Footprints:SW_Hotswap_Kailh_Choc_V1V2_THT
- DOWN1: footprint moth footprints:SW_Gateron_LowProfile_HotSwap_THT -> Box Footprints:SW_Hotswap_Kailh_Choc_V1V2
- J4, J5: footprint moth footprints:FPC-05F-30PH20 -> Box Footprints:FPC-05F-30PH20
- U2: footprint footprint:FPC-SMD_X05A26H12G -> Box Dependecies:FPC-SMD_X05A26H12G
- U3: footprint qw-footprints:RP2040-QFN-56 -> Box Footprints:RP2040-QFN-56
- moved R5 8.97 mm to (225.8, 127.7)
- moved C10 8.97 mm to (228.5, 117.2)
- moved C12 8.97 mm to (226.7, 121.0)
- moved C13 8.97 mm to (224.2, 112.0)
- moved C2 8.97 mm to (236.8, 121.5)
- moved C3 8.97 mm to (233.7, 113.7)
- moved C4 8.97 mm to (226.7, 120.0)
- moved C5 8.97 mm to (228.5, 115.7)
- moved C7 8.97 mm to (209.1, 111.5)
- moved C8 8.97 mm to (209.3, 118.2)
- moved C9 8.97 mm to (229.9, 124.5)
- moved J1 8.97 mm to (247.0, 106.9)
- moved MX1 8.97 mm to (185.1, 130.3)
- moved R6 8.97 mm to (225.8, 129.2)
- moved R7 8.97 mm to (213.4, 123.1)
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Routing:
- net GND: track 78.8 -> 102.1 mm
- net C_LT: track 74.1 -> 51.8 mm, vias 1 -> 2
- net 3vDiode: track 142.2 -> 163.5 mm
- net (no net): track 0.00 -> 18.4 mm
- net C_DN: track 89.4 -> 75.3 mm, vias 1 -> 2
- net M1: track 66.1 -> 52.8 mm
- net M2: track 91.0 -> 78.3 mm
- net C_RT: track 68.8 -> 56.1 mm
- net C_UP: track 51.1 -> 39.9 mm
- net Z: track 82.0 -> 71.1 mm
- net A: track 84.2 -> 73.5 mm
- net UP: track 103.2 -> 108.8 mm
- net X: track 48.6 -> 43.1 mm
- net Y: track 54.0 -> 57.5 mm, vias 0 -> 2
- net RIGHT: track 57.6 -> 54.7 mm
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Other:
- board text added: "THE MOTH BY RANA LABS - PCB by campagne"
- board text removed: "A"
- board text removed: "B"
- board text removed: "C-DOWN"
- board text removed: "C-LEFT"
- board text removed: "C-RIGHT"
- board text removed: "C-UP"
- board text removed: "DOWN"
- board text removed: "L"
- board text removed: "LEFT"
- board text removed: "LS"
- board text removed: "MS"
- board text removed: "MX"
- board text removed: "MY"
- board text removed: "R"
- board text removed: "RANA MOTH BY RANA LABS"
- board text removed: "RIGHT"
- board text removed: "START"
- board text removed: "UP"
- board text removed: "X"
- board text removed: "Y"
- board text removed: "Z"

Commit message: Add files via upload
Parts:
- renumbered A1 to A, B1 to B, C_DOWN1 to C_DOWN, C_LEFT1 to C_LEFT, C_RIGHT1 to C_RIGHT, C_UP1 to C_UP, DOWN1 to DOWN, L1 to L, LEFT1 to LEFT, LS1 to LS, MS1 to MS, MX1 to MX, MY1 to MY, R1 to R, RIGHT1 to RIGHT, START1 to START, UP1 to UP, X1 to X, Y2 to Y, Z1 to Z
Routing:
- net (no net): track 18.4 -> 0.00 mm
- net B: track 26.1 -> 20.2 mm
- net UP: track 108.8 -> 105.9 mm
- net GND: track 102.1 -> 103.2 mm
Other:
- board text added: "+5V"
- board text added: "3v3"
- board text added: "A"
- board text added: "B"
- board text added: "C_DOWN"
- board text added: "C_LEFT"
- board text added: "C_RIGHT"
- board text added: "C_UP"
- board text added: "D+"
- board text added: "D-"
- board text added: "DATA"
- board text added: "DOWN"
- board text added: "GND"
- board text added: "L"
- board text added: "LEFT"
- board text added: "LS"
- board text added: "MS"
- board text added: "MX"
- board text added: "MY"
- board text added: "R"
- board text added: "RIGHT"
- board text added: "START"
- board text added: "UP"
- board text added: "X"
- board text added: "Y"
- board text added: "Z"
- board text removed: "3v3 DATA D- D+ 5+ GND"

Commit message: PCB files possibly done pending testing
Parts:
- moved MX1 119.8 mm to (65.2, 129.8)
- moved J4 117.2 mm to (46.1, 79.3)
- moved C10 117.2 mm to (111.3, 117.8)
- moved C12 117.2 mm to (109.5, 121.6)
- moved C13 117.2 mm to (106.9, 112.6)
- moved C2 117.2 mm to (119.6, 122.2)
- moved C3 117.2 mm to (116.5, 114.4)
- moved C4 117.2 mm to (109.5, 120.6)
- moved C5 117.2 mm to (111.3, 116.3)
- moved C7 117.2 mm to (91.8, 112.1)
- moved C8 117.2 mm to (92.1, 118.8)
- moved C9 117.2 mm to (112.7, 125.2)
- moved J1 117.2 mm to (129.8, 107.6)
- moved L1 117.2 mm to (133.5, 74.6)
- moved R5 117.2 mm to (108.5, 128.3)
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- renumbered A to A1, B to B1, C_DOWN to C_DOWN1, C_LEFT to C_LEFT1, C_RIGHT to C_RIGHT1, C_UP to C_UP1, DOWN to DOWN1, L to L1, LEFT to LEFT1, LS to LS1, MS to MS1, MX to MX1, MY to MY1, R to R1, RIGHT to RIGHT1, START to START1, UP to UP1, X to X1, Y to Y2, Z to Z1
Routing:
- net GND: track 103.2 -> 76.0 mm
- net A RIBBON: track 91.5 -> 80.8 mm
- net C_LT RIBBON: track 91.6 -> 81.0 mm
- net C_DN RIBBON: track 91.3 -> 81.5 mm
- net DATA: track 92.7 -> 102.5 mm
- net C_UP RIBBON: track 91.5 -> 82.8 mm
- net M1: track 52.8 -> 58.8 mm
- net L: track 72.7 -> 76.6 mm
- net R: track 33.8 -> 37.7 mm, vias 0 -> 2
- net MS RIBBON: track 110.2 -> 113.0 mm
- net M2: track 78.3 -> 81.1 mm
- net C_RT RIBBON: track 111.3 -> 113.9 mm
- net UP RIBBON: track 110.8 -> 113.4 mm
- net Z RIBBON: track 111.0 -> 113.6 mm
- net LS RIBBON: track 111.7 -> 114.2 mm
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Other:
- board size 220.6 x 118.4 mm -> 210.2 x 119.7 mm
- board text added: "The Moth by Rana Labs - PCB by campagne"
- board text removed: "THE MOTH BY RANA LABS - PCB by campagne"

Commit message: Add files via upload
Parts:
- DOWN1: footprint Box Footprints:SW_Hotswap_Kailh_Choc_V1V2 -> Box Footprints:SW_Hotswap_Kailh_Choc_V1V2_THT
- moved MX1 1.56 mm to (66.6, 129.1)
Routing:
- net GND: track 76.0 -> 62.3 mm
- net M1: track 58.8 -> 58.0 mm
- net DATA: track 102.5 -> 103.1 mm
Changed lines of the file:
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@@
 	(footprint "Box Footprints:SW_Hotswap_Kailh_Choc_V1V2_THT"
 		(layer "B.Cu")
-		(at 65.248497 129.753866 180)
+		(at 66.64 129.05 180)
 		(descr "Kailh Choc keyswitch CPG1350 V1 CPG1353 V2 Hotswap")
 		(tags "Kailh Choc Keyswitch Switch CPG1350 V1 CPG1353 V2 Hotswap Cutout")
@@
 		)
 	)
-	(footprint "Box Footprints:SW_Hotswap_Kailh_Choc_V1V2"
+	(footprint "Box Footprints:SW_Hotswap_Kailh_Choc_V1V2_THT"
 		(layer "B.Cu")
 		(at 89.806 73.058 180)
@@
 		(tags "Kailh Choc Keyswitch Switch CPG1350 V1 CPG1353 V2 Hotswap Cutout")
 		(property "Reference" "DOWN1"
-			(at 0.04 -9.082934 0)
+			(at 0 9 0)
 			(layer "B.SilkS")
 			(effects
@@
 			)
 		)
-		(property "Footprint" "Box Footprints:SW_Hotswap_Kailh_Choc_V1V2"
+		(property "Footprint" "Box Footprints:SW_Hotswap_Kailh_Choc_V1V2_THT"
 			(at 0 0 0)
 			(layer "B.Fab")
@@
 		(sheetname "Root")
 		(sheetfile "Moth.kicad_sch")
-		(attr smd)
+		(attr through_hole)
 		(fp_line
 			(start 7.6 7.6)
@@
 			(layers "*.Cu" "*.Mask")
 		)
-		(pad "1" smd roundrect
+		(pad "1" thru_hole circle
+			(at -4.235 5.17 180)
+			(size 0.4 0.4)
+			(drill 0.3)
+			(layers "*.Cu" "*.Mask")
+			(remove_unused_layers no)
+			(net 25 "DOWN")
+			(pinfunction "1")
+			(pintype "passive")
+		)
+		(pad "1" thru_hole circle
+			(at -4.235 6.75 180)
+			(size 0.4 0.4)
+			(drill 0.3)
+			(layers "*.Cu" "*.Mask")
+			(remove_unused_layers no)
+			(net 25 "DOWN")
+			(pinfunction "1")
+			(pintype "passive")
+		)
+		(pad "1" thru_hole circle
 			(at -3.5 6 180)
-			(size 2.55 2.5)
+			(size 0.4 0.4)
+			(drill 0.3)
+			(layers "*.Cu" "*.Mask")
+			(remove_unused_layers no)
+			(net 25 "DOWN")
+			(pinfunction "1")
+			(pintype "passive")
+		)
+		(pad "1" smd roundrect
+			(at -3.475 6 180)
+			(size 2.55 2.55)
 			(layers "F.Cu" "F.Paste" "F.Mask")
 			(roundrect_rratio 0.1)
@@
 			(pintype "passive")
 		)
+		(pad "1" thru_hole circle
+			(at -2.805 5.13 180)
+			(size 0.4 0.4)
+			(drill 0.3)
+			(layers "*.Cu" "*.Mask")
+			(remove_unused_layers no)
+			(net 25 "DOWN")
+			(pinfunction "1")
+			(pintype "passive")
+		)
+		(pad "1" thru_hole circle
+			(at -2.805 6.75 180)
+			(size 0.4 0.4)
+			(drill 0.3)
+			(layers "*.Cu" "*.Mask")
+			(remove_unused_layers no)
+			(net 25 "DOWN")
+			(pinfunction "1")
+			(pintype "passive")
+		)
+		(pad "2" thru_hole circle
+			(at 7.807306 2.964485 180)
+			(size 0.4 0.4)
+			(drill 0.3)
+			(layers "*.Cu" "*.Mask")
+			(remove_unused_layers no)
+			(net 1 "GND")
+			(pinfunction "2")
+			(pintype "passive")
+		)
+		(pad "2" thru_hole circle
+			(at 7.807306 4.544485 180)
+			(size 0.4 0.4)
+			(drill 0.3)
+			(layers "*.Cu" "*.Mask")
+			(remove_unused_layers no)
+			(net 1 "GND")
+			(pinfunction "2")
+			(pintype "passive")
+		)
 		(pad "2" smd roundrect
-			(at 8.5 3.8 180)
-			(size 2.55 2.5)
+			(at 8.512306 3.774485 180)
+			(size 2.55 2.55)
 			(layers "F.Cu" "F.Paste" "F.Mask")
 			(roundrect_rratio 0.1)
@@
 			(pintype "passive")
 		)
+		(pad "2" thru_hole circle
+			(at 8.542306 3.794485 180)
+			(size 0.4 0.4)
+			(drill 0.3)
+			(layers "*.Cu" "*.Mask")
+			(remove_unused_layers no)
+			(net 1 "GND")
+			(pinfunction "2")
+			(pintype "passive")
+		)
+		(pad "2" thru_hole circle
+			(at 9.237306 2.924485 180)
+			(size 0.4 0.4)
+			(drill 0.3)
+			(layers "*.Cu" "*.Mask")
+			(remove_unused_layers no)
+			(net 1 "GND")
+			(pinfunction "2")
+			(pintype "passive")
+		)
+		(pad "2" thru_hole circle
+			(at 9.237306 4.544485 180)
+			(size 0.4 0.4)
+			(drill 0.3)
+			(layers "*.Cu" "*.Mask")
+			(remove_unused_layers no)
+			(net 1 "GND")
+			(pinfunction "2")
+			(pintype "passive")
+		)
 		(model "${KICAD6_3RD_PARTY}/3dmodels/com_github_perigoso_keyswitch-kicad-library/3d-library.3dshapes/SW_Hotswap_Kailh_Choc_V1.wrl"
 			(offset
@@
 		(tags "Kailh Choc Keyswitch Switch CPG1350 V1 CPG1353 V2 Hotswap Cutout")
 		(property "Reference" "L1"
-			(at -0.0043 -8.987436 0)
+			(at 0 9 0)
 			(layer "B.SilkS")
 			(effects
@@
 		(tags "Kailh Choc Keyswitch Switch CPG1350 V1 CPG1353 V2 Hotswap Cutout")
 		(property "Reference" "LEFT1"
-			(at -0.229253 -8.938295 0)
+			(at 0 9 0)
 			(layer "B.SilkS")
 			(effects
@@
 		(tags "Kailh Choc Keyswitch Switch CPG1350 V1 CPG1353 V2 Hotswap Cutout")
 		(property "Reference" "A1"
-			(at -0.078886 9.502429 0)
+			(at 0 9 0)
 			(layer "B.SilkS")
 			(effects
@@
 		(tags "Kailh Choc Keyswitch Switch CPG1350 V1 CPG1353 V2 Hotswap Cutout")
 		(property "Reference" "MY1"
-			(at 0 9.21425 0)
+			(at 0 9 0)
 			(layer "B.SilkS")
 			(effects
@@
 		(tags "Kailh Choc Keyswitch Switch CPG1350 V1 CPG1353 V2 Hotswap Cutout")
 		(property "Reference" "RIGHT1"
-			(at -0.026958 -8.904533 0)
+			(at 0 9 0)
 			(layer "B.SilkS")
 			(effects
@@
 	)
 	(gr_text "MX"
-		(at 77.266 130.890934 -0)
+		(at 75.05 130.96 -0)
 		(layer "F.SilkS")
 		(effects
@@
 	)
 	(segment
-		(start 118.766 85.890934)
-		(end 116.516 88.140934)
-		(width 0.25)
-		(layer "B.Cu")
-		(net 1)
-	)
-	(segment
 		(start 101.966489 116.568566)
 		(end 104.516489 116.568566)
@@
 	)
 	(segment
-		(start 129.266 85.890934)
-		(end 118.766 85.890934)
-		(width 0.25)
-		(layer "B.Cu")
-		(net 1)
-	)
-	(segment
 		(start 104.516489 117.843566)
 		(end 101.966489 117.843566)
@@
 	)
 	(segment
-		(start 109.80913 128.492041)
-		(end 109.80913 130.303566)
+		(start 105.009 81.911)
+		(end 105.009 81.714298)
 		(width 0.25)
 		(layer "B.Cu")
@@
 	)
 	(segment
-		(start 105.3 82.202)
-		(end 105.009 81.911)
+		(start 101.186 77.891298)
+		(end 101.186 72.028824)
 		(width 0.25)
 		(layer "B.Cu")
@@
 	)
 	(segment
-		(start 101.186 73.008)
-		(end 91.076 62.898)
+		(start 101.186 72.028824)
+		(end 93.957176 64.8)
 		(width 0.25)
 		(layer "B.Cu")
@@
 	)
 	(segment
-		(start 116.222 108.11)
-		(end 116.222 115.264171)
+		(start 109.80913 128.492041)
+		(end 109.80913 130.303566)
 		(width 0.25)
 		(layer "B.Cu")
@@
 	)
 	(segment
-		(start 101.266 91.890934)
-		(end 101.266 93.154)
+		(start 116.222 108.11)
+		(end 116.222 115.264171)
 		(width 0.25)
 		(layer "B.Cu")
@@
 	)
 	(segment
-		(start 101.186 77.891298)
-		(end 101.186 73.008)
+		(start 101.266 91.890934)
+		(end 101.266 93.154)
 		(width 0.25)
 		(layer "B.Cu")
@@
 	)
 	(segment
-		(start 115.881489 122.419682)
-		(end 109.80913 128.492041)
+		(start 93.957176 64.8)
+		(end 92.47 64.8)
 		(width 0.25)
 		(layer "B.Cu")
@@
 	)
 	(segment
-		(start 91.076 62.898)
-		(end 90.568 62.898)
+		(start 115.881489 122.419682)
+		(end 109.80913 128.492041)
 		(width 0.25)
 		(layer "B.Cu")
@@
 	)
 	(segment
-		(start 105.009 81.911)
-		(end 105.009 81.714298)
+		(start 105.009 81.714298)
+		(end 101.186 77.891298)
 		(width 0.25)
 		(layer "B.Cu")
@@
 	)
 	(segment
-		(start 105.009 81.714298)
-		(end 101.186 77.891298)
+		(start 92.47 64.8)
+		(end 90.568 62.898)
 		(width 0.25)
 		(layer "B.Cu")
@@
 		(net 8)
 	)
+	(segment
+		(start 105.3 82.202)
+		(end 105.009 81.911)
+		(width 0.25)
+		(layer "B.Cu")
+		(net 8)
+	)
 	(arc
 		(start 107.186088 128.923165)
@@
 	)
 	(segment
-		(start 68.664934 123.695303)
-		(end 68.723497 123.753866)
+		(start 70.115 121.802841)
+		(end 70.115 122.362363)
 		(width 0.2)
 		(layer "F.Cu")
@@
 	(segment
 		(start 68.664934 120.352775)
-		(end 68.664934 123.695303)
+		(end 70.115 121.802841)
 		(width 0.2)
 		(layer "F.Cu")
